File: 3V3-LDO.sch (KiCad schematic (older format))
At the start: 5 parts, among them U2 SSP6206

Commit message: Updated copper pours to avoid short between V_USB and GND
Parts:
- C6, C9: Mfr Part # (none) -> CL10B105KQ8NNNC; Supplier (none) -> LCSC; Supplier Part # (none) -> C105524
Changed lines of the file:
@@
 F 2 "Capacitor_SMD:C_0603_1608Metric" H 6400 3750 50  0001 C CNN
 F 3 "~" H 6400 3750 50  0001 C CNN
+F 4 "CL10B105KQ8NNNC" H 6400 3750 50  0001 C CNN "Mfr Part #"
+F 5 "LCSC" H 6400 3750 50  0001 C CNN "Supplier"
+F 6 "C105524" H 6400 3750 50  0001 C CNN "Supplier Part #"
 	1    6400 3750
 	1    0    0    -1
@@
 F 2 "Capacitor_SMD:C_0603_1608Metric" H 4200 3750 50  0001 C CNN
 F 3 "~" H 4200 3750 50  0001 C CNN
+F 4 "CL10B105KQ8NNNC" H 4200 3750 50  0001 C CNN "Mfr Part #"
+F 5 "LCSC" H 4200 3750 50  0001 C CNN "Supplier"
+F 6 "C105524" H 4200 3750 50  0001 C CNN "Supplier Part #"
 	1    4200 3750
 	-1   0    0    -1
