File: Addressable_LEDs.sch (KiCad schematic (older format))
At the start: 24 parts

Commit message: Updated copper pours to avoid short between V_USB and GND
Parts:
- C10, C11, C12, C13, C14, C15, C16, C17, C18, C19, C20, C21: Mfr Part # (none) -> 0603F104Z160CT; Supplier (none) -> LCSC; Supplier Part # (none) -> C387984
- D10, D11, D12, D13, D14, D15, D4, D5, D6, D7, D8, D9: Mfr Part # (none) -> WS2812E; Supplier (none) -> LCSC; Supplier Part # (none) -> C139127
Changed lines of the file:
@@
 F 2 "LED_SMD:LED_WS2812B_PLCC4_5.0x5.0mm_P3.2mm" H 1950 1750 50  0001 L TNN
 F 3 "https://cdn-shop.adafruit.com/datasheets/WS2812B.pdf" H 2000 1675 50  0001 L TNN
+F 4 "WS2812E" H 1900 2050 50  0001 C CNN "Mfr Part #"
+F 5 "LCSC" H 1900 2050 50  0001 C CNN "Supplier"
+F 6 "C139127" H 1900 2050 50  0001 C CNN "Supplier Part #"
 	1    1900 2050
 	1    0    0    -1
@@
 F 2 "Capacitor_SMD:C_0603_1608Metric" H 1938 3000 50  0001 C CNN
 F 3 "~" H 1900 3150 50  0001 C CNN
+F 4 "0603F104Z160CT" H 1900 3150 50  0001 C CNN "Mfr Part #"
+F 5 "LCSC" H 1900 3150 50  0001 C CNN "Supplier"
+F 6 "C387984" H 1900 3150 50  0001 C CNN "Supplier Part #"
 	1    1900 3150
 	1    0    0    -1
@@
 F 2 "LED_SMD:LED_WS2812B_PLCC4_5.0x5.0mm_P3.2mm" H 3300 1750 50  0001 L TNN
 F 3 "https://cdn-shop.adafruit.com/datasheets/WS2812B.pdf" H 3350 1675 50  0001 L TNN
+F 4 "WS2812E" H 3250 2050 50  0001 C CNN "Mfr Part #"
+F 5 "LCSC" H 3250 2050 50  0001 C CNN "Supplier"
+F 6 "C139127" H 3250 2050 50  0001 C CNN "Supplier Part #"
 	1    3250 2050
 	1    0    0    -1
@@
 F 2 "Capacitor_SMD:C_0603_1608Metric" H 3288 3000 50  0001 C CNN
 F 3 "~" H 3250 3150 50  0001 C CNN
+F 4 "0603F104Z160CT" H 3250 3150 50  0001 C CNN "Mfr Part #"
+F 5 "LCSC" H 3250 3150 50  0001 C CNN "Supplier"
+F 6 "C387984" H 3250 3150 50  0001 C CNN "Supplier Part #"
 	1    3250 3150
 	1    0    0    -1
@@
 F 2 "LED_SMD:LED_WS2812B_PLCC4_5.0x5.0mm_P3.2mm" H 4650 1750 50  0001 L TNN
 F 3 "https://cdn-shop.adafruit.com/datasheets/WS2812B.pdf" H 4700 1675 50  0001 L TNN
+F 4 "WS2812E" H 4600 2050 50  0001 C CNN "Mfr Part #"
+F 5 "LCSC" H 4600 2050 50  0001 C CNN "Supplier"
+F 6 "C139127" H 4600 2050 50  0001 C CNN "Supplier Part #"
 	1    4600 2050
 	1    0    0    -1
@@
 F 2 "Capacitor_SMD:C_0603_1608Metric" H 4638 3000 50  0001 C CNN
 F 3 "~" H 4600 3150 50  0001 C CNN
+F 4 "0603F104Z160CT" H 4600 3150 50  0001 C CNN "Mfr Part #"
+F 5 "LCSC" H 4600 3150 50  0001 C CNN "Supplier"
+F 6 "C387984" H 4600 3150 50  0001 C CNN "Supplier Part #"
 	1    4600 3150
 	1    0    0    -1
@@
 F 2 "LED_SMD:LED_WS2812B_PLCC4_5.0x5.0mm_P3.2mm" H 6000 1750 50  0001 L TNN
 F 3 "https://cdn-shop.adafruit.com/datasheets/WS2812B.pdf" H 6050 1675 50  0001 L TNN
+F 4 "WS2812E" H 5950 2050 50  0001 C CNN "Mfr Part #"
+F 5 "LCSC" H 5950 2050 50  0001 C CNN "Supplier"
+F 6 "C139127" H 5950 2050 50  0001 C CNN "Supplier Part #"
 	1    5950 2050
 	1    0    0    -1
@@
 F 2 "Capacitor_SMD:C_0603_1608Metric" H 5988 3000 50  0001 C CNN
 F 3 "~" H 5950 3150 50  0001 C CNN
+F 4 "0603F104Z160CT" H 5950 3150 50  0001 C CNN "Mfr Part #"
+F 5 "LCSC" H 5950 3150 50  0001 C CNN "Supplier"
+F 6 "C387984" H 5950 3150 50  0001 C CNN "Supplier Part #"
 	1    5950 3150
 	1    0    0    -1
@@
 F 2 "LED_SMD:LED_WS2812B_PLCC4_5.0x5.0mm_P3.2mm" H 7350 1750 50  0001 L TNN
 F 3 "https://cdn-shop.adafruit.com/datasheets/WS2812B.pdf" H 7400 1675 50  0001 L TNN
+F 4 "WS2812E" H 7300 2050 50  0001 C CNN "Mfr Part #"
+F 5 "LCSC" H 7300 2050 50  0001 C CNN "Supplier"
+F 6 "C139127" H 7300 2050 50  0001 C CNN "Supplier Part #"
 	1    7300 2050
 	1    0    0    -1
@@
 F 2 "Capacitor_SMD:C_0603_1608Metric" H 7338 3000 50  0001 C CNN
 F 3 "~" H 7300 3150 50  0001 C CNN
+F 4 "0603F104Z160CT" H 7300 3150 50  0001 C CNN "Mfr Part #"
+F 5 "LCSC" H 7300 3150 50  0001 C CNN "Supplier"
+F 6 "C387984" H 7300 3150 50  0001 C CNN "Supplier Part #"
 	1    7300 3150
 	1    0    0    -1
@@
 F 2 "LED_SMD:LED_WS2812B_PLCC4_5.0x5.0mm_P3.2mm" H 8700 1750 50  0001 L TNN
 F 3 "https://cdn-shop.adafruit.com/datasheets/WS2812B.pdf" H 8750 1675 50  0001 L TNN
+F 4 "WS2812E" H 8650 2050 50  0001 C CNN "Mfr Part #"
+F 5 "LCSC" H 8650 2050 50  0001 C CNN "Supplier"
+F 6 "C139127" H 8650 2050 50  0001 C CNN "Supplier Part #"
 	1    8650 2050
 	1    0    0    -1
@@
 F 2 "Capacitor_SMD:C_0603_1608Metric" H 8688 3000 50  0001 C CNN
 F 3 "~" H 8650 3150 50  0001 C CNN
+F 4 "0603F104Z160CT" H 8650 3150 50  0001 C CNN "Mfr Part #"
+F 5 "LCSC" H 8650 3150 50  0001 C CNN "Supplier"
+F 6 "C387984" H 8650 3150 50  0001 C CNN "Supplier Part #"
 	1    8650 3150
 	1    0    0    -1
@@
 F 2 "LED_SMD:LED_WS2812B_PLCC4_5.0x5.0mm_P3.2mm" H 1950 4400 50  0001 L TNN
 F 3 "https://cdn-shop.adafruit.com/datasheets/WS2812B.pdf" H 2000 4325 50  0001 L TNN
+F 4 "WS2812E" H 1900 4700 50  0001 C CNN "Mfr Part #"
+F 5 "LCSC" H 1900 4700 50  0001 C CNN "Supplier"
+F 6 "C139127" H 1900 4700 50  0001 C CNN "Supplier Part #"
 	1    1900 4700
 	1    0    0    -1
@@
 F 2 "Capacitor_SMD:C_0603_1608Metric" H 1938 5650 50  0001 C CNN
 F 3 "~" H 1900 5800 50  0001 C CNN
+F 4 "0603F104Z160CT" H 1900 5800 50  0001 C CNN "Mfr Part #"
+F 5 "LCSC" H 1900 5800 50  0001 C CNN "Supplier"
+F 6 "C387984" H 1900 5800 50  0001 C CNN "Supplier Part #"
 	1    1900 5800
 	1    0    0    -1
@@
 F 2 "LED_SMD:LED_WS2812B_PLCC4_5.0x5.0mm_P3.2mm" H 3300 4400 50  0001 L TNN
 F 3 "https://cdn-shop.adafruit.com/datasheets/WS2812B.pdf" H 3350 4325 50  0001 L TNN
+F 4 "WS2812E" H 3250 4700 50  0001 C CNN "Mfr Part #"
+F 5 "LCSC" H 3250 4700 50  0001 C CNN "Supplier"
+F 6 "C139127" H 3250 4700 50  0001 C CNN "Supplier Part #"
 	1    3250 4700
 	1    0    0    -1
@@
 F 2 "Capacitor_SMD:C_0603_1608Metric" H 3288 5650 50  0001 C CNN
 F 3 "~" H 3250 5800 50  0001 C CNN
+F 4 "0603F104Z160CT" H 3250 5800 50  0001 C CNN "Mfr Part #"
+F 5 "LCSC" H 3250 5800 50  0001 C CNN "Supplier"
+F 6 "C387984" H 3250 5800 50  0001 C CNN "Supplier Part #"
 	1    3250 5800
 	1    0    0    -1
@@
 F 2 "LED_SMD:LED_WS2812B_PLCC4_5.0x5.0mm_P3.2mm" H 4650 4400 50  0001 L TNN
 F 3 "https://cdn-shop.adafruit.com/datasheets/WS2812B.pdf" H 4700 4325 50  0001 L TNN
+F 4 "WS2812E" H 4600 4700 50  0001 C CNN "Mfr Part #"
+F 5 "LCSC" H 4600 4700 50  0001 C CNN "Supplier"
+F 6 "C139127" H 4600 4700 50  0001 C CNN "Supplier Part #"
 	1    4600 4700
 	1    0    0    -1
@@
 F 2 "Capacitor_SMD:C_0603_1608Metric" H 4638 5650 50  0001 C CNN
 F 3 "~" H 4600 5800 50  0001 C CNN
+F 4 "0603F104Z160CT" H 4600 5800 50  0001 C CNN "Mfr Part #"
+F 5 "LCSC" H 4600 5800 50  0001 C CNN "Supplier"
+F 6 "C387984" H 4600 5800 50  0001 C CNN "Supplier Part #"
 	1    4600 5800
 	1    0    0    -1
@@
 F 2 "LED_SMD:LED_WS2812B_PLCC4_5.0x5.0mm_P3.2mm" H 6000 4400 50  0001 L TNN
 F 3 "https://cdn-shop.adafruit.com/datasheets/WS2812B.pdf" H 6050 4325 50  0001 L TNN
+F 4 "WS2812E" H 5950 4700 50  0001 C CNN "Mfr Part #"
+F 5 "LCSC" H 5950 4700 50  0001 C CNN "Supplier"
+F 6 "C139127" H 5950 4700 50  0001 C CNN "Supplier Part #"
 	1    5950 4700
 	1    0    0    -1
@@
 F 2 "Capacitor_SMD:C_0603_1608Metric" H 5988 5650 50  0001 C CNN
 F 3 "~" H 5950 5800 50  0001 C CNN
+F 4 "0603F104Z160CT" H 5950 5800 50  0001 C CNN "Mfr Part #"
+F 5 "LCSC" H 5950 5800 50  0001 C CNN "Supplier"
+F 6 "C387984" H 5950 5800 50  0001 C CNN "Supplier Part #"
 	1    5950 5800
 	1    0    0    -1
@@
 F 2 "LED_SMD:LED_WS2812B_PLCC4_5.0x5.0mm_P3.2mm" H 7350 4400 50  0001 L TNN
 F 3 "https://cdn-shop.adafruit.com/datasheets/WS2812B.pdf" H 7400 4325 50  0001 L TNN
+F 4 "WS2812E" H 7300 4700 50  0001 C CNN "Mfr Part #"
+F 5 "LCSC" H 7300 4700 50  0001 C CNN "Supplier"
+F 6 "C139127" H 7300 4700 50  0001 C CNN "Supplier Part #"
 	1    7300 4700
 	1    0    0    -1
@@
 F 2 "Capacitor_SMD:C_0603_1608Metric" H 7338 5650 50  0001 C CNN
 F 3 "~" H 7300 5800 50  0001 C CNN
+F 4 "0603F104Z160CT" H 7300 5800 50  0001 C CNN "Mfr Part #"
+F 5 "LCSC" H 7300 5800 50  0001 C CNN "Supplier"
+F 6 "C387984" H 7300 5800 50  0001 C CNN "Supplier Part #"
 	1    7300 5800
 	1    0    0    -1
@@
 F 2 "LED_SMD:LED_WS2812B_PLCC4_5.0x5.0mm_P3.2mm" H 8700 4400 50  0001 L TNN
 F 3 "https://cdn-shop.adafruit.com/datasheets/WS2812B.pdf" H 8750 4325 50  0001 L TNN
+F 4 "WS2812E" H 8650 4700 50  0001 C CNN "Mfr Part #"
+F 5 "LCSC" H 8650 4700 50  0001 C CNN "Supplier"
+F 6 "C139127" H 8650 4700 50  0001 C CNN "Supplier Part #"
 	1    8650 4700
 	1    0    0    -1
@@
 F 2 "Capacitor_SMD:C_0603_1608Metric" H 8688 5650 50  0001 C CNN
 F 3 "~" H 8650 5800 50  0001 C CNN
+F 4 "0603F104Z160CT" H 8650 5800 50  0001 C CNN "Mfr Part #"
+F 5 "LCSC" H 8650 5800 50  0001 C CNN "Supplier"
+F 6 "C387984" H 8650 5800 50  0001 C CNN "Supplier Part #"
 	1    8650 5800
 	1    0    0    -1
