File: STM32F030F4Px.sch (KiCad schematic (older format))
At the start: 8 parts, among them U1 STM32F030F4Px

Commit message: Updated copper pours to avoid short between V_USB and GND
Parts:
- C3, C4: Mfr Part # (none) -> 0603F104Z160CT; Supplier (none) -> LCSC; Supplier Part # (none) -> C387984
- U1: Mfr Part # (none) -> STM32F030F4P6; Supplier (none) -> LCSC; Supplier Part # (none) -> C32908
Changed lines of the file:
@@
 F 2 "Package_SO:TSSOP-20_4.4x6.5mm_P0.65mm" H 5100 2750 50  0001 R CNN
 F 3 "http://www.st.com/st-web-ui/static/active/en/resource/technical/document/datasheet/DM00088500.pdf" H 5500 3450 50  0001 C CNN
+F 4 "STM32F030F4P6" H 5500 3450 50  0001 C CNN "Mfr Part #"
+F 5 "LCSC" H 5500 3450 50  0001 C CNN "Supplier"
+F 6 "C32908" H 5500 3450 50  0001 C CNN "Supplier Part #"
 	1    5500 3450
 	1    0    0    -1
@@
 F 2 "Capacitor_SMD:C_0603_1608Metric" H 1638 4400 50  0001 C CNN
 F 3 "~" H 1600 4550 50  0001 C CNN
+F 4 "0603F104Z160CT" H 1600 4550 50  0001 C CNN "Mfr Part #"
+F 5 "LCSC" H 1600 4550 50  0001 C CNN "Supplier"
+F 6 "C387984" H 1600 4550 50  0001 C CNN "Supplier Part #"
 	1    1600 4550
 	1    0    0    -1
@@
 F 2 "Capacitor_SMD:C_0603_1608Metric" H 938 3950 50  0001 C CNN
 F 3 "~" H 900 4100 50  0001 C CNN
+F 4 "0603F104Z160CT" H 900 4100 50  0001 C CNN "Mfr Part #"
+F 5 "LCSC" H 900 4100 50  0001 C CNN "Supplier"
+F 6 "C387984" H 900 4100 50  0001 C CNN "Supplier Part #"
 	1    900  4100
 	1    0    0    -1
